File: offroad-cpu-hardware.sch (EAGLE design)
At the start: 15 parts, among them IC1 ATmega328-DIP-Prgrammed, Q1 2N3904, U1 LCD-16X2NOHOLES, Y1 16MHz

Commit message: Removes timing crystal and associated capacitors
http://arduino.cc/en/Tutorial/ArduinoToBreadboard
Parts:
- removed C1, C2: 22pF, SparkFun:CAPPTH2
- removed Y1: 16MHz, SparkFun:CRYSTALHC49US
Connections:
- removed net XTAL1: C2.1, IC1.PB6(XTAL1/TOSC1), Y1.2
- removed net XTAL2: C1.1, IC1.PB7(XTAL2/TOSC2), Y1.1
- net GND: no longer C1.2, C2.2
Changed lines of the file:
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@@
 <?xml version="1.0" encoding="utf-8"?>
 <!DOCTYPE eagle SYSTEM "eagle.dtd">
-<eagle version="6.4">
+<eagle version="7.2.0">
 <drawing>
 <settings>
@@
 <part name="GND1" library="SparkFun" deviceset="GND" device=""/>
 <part name="U$6" library="SparkFun" deviceset="5V" device=""/>
-<part name="Y1" library="SparkFun" deviceset="CRYSTAL" device="HC49US" value="16MHz"/>
-<part name="C1" library="SparkFun" deviceset="CAP" device="PTH2" value="22pF"/>
-<part name="C2" library="SparkFun" deviceset="CAP" device="PTH2" value="22pF"/>
-<part name="GND3" library="SparkFun" deviceset="GND" device=""/>
 <part name="GND4" library="SparkFun" deviceset="GND" device=""/>
 <part name="U1" library="SparkFun-Displays" deviceset="LCD-16X2" device="NOHOLES" value="LCD-16X2NOHOLES"/>
@@
 <instance part="GND1" gate="1" x="99.06" y="83.82"/>
 <instance part="U$6" gate="G$1" x="99.06" y="106.68"/>
-<instance part="Y1" gate="G$1" x="93.98" y="114.3" rot="R90"/>
-<instance part="C1" gate="G$1" x="91.44" y="104.14"/>
-<instance part="C2" gate="G$1" x="81.28" y="104.14"/>
-<instance part="GND3" gate="1" x="86.36" y="93.98"/>
 <instance part="GND4" gate="1" x="27.94" y="137.16"/>
 <instance part="U1" gate="G$1" x="20.32" y="73.66" smashed="yes" rot="R180">
@@
 </segment>
 <segment>
-<wire x1="81.28" y1="101.6" x2="81.28" y2="99.06" width="0.1524" layer="91"/>
-<wire x1="81.28" y1="99.06" x2="86.36" y2="99.06" width="0.1524" layer="91"/>
-<wire x1="86.36" y1="99.06" x2="91.44" y2="99.06" width="0.1524" layer="91"/>
-<wire x1="91.44" y1="99.06" x2="91.44" y2="101.6" width="0.1524" layer="91"/>
-<wire x1="86.36" y1="96.52" x2="86.36" y2="99.06" width="0.1524" layer="91"/>
-<junction x="86.36" y="99.06"/>
-<pinref part="C2" gate="G$1" pin="2"/>
-<pinref part="C1" gate="G$1" pin="2"/>
-<pinref part="GND3" gate="1" pin="GND"/>
-</segment>
-<segment>
 <wire x1="30.48" y1="53.34" x2="33.02" y2="53.34" width="0.1524" layer="91"/>
 <wire x1="33.02" y1="53.34" x2="33.02" y2="50.8" width="0.1524" layer="91"/>
@@
 </segment>
 </net>
-<net name="XTAL1" class="0">
-<segment>
-<wire x1="101.6" y1="116.84" x2="93.98" y2="116.84" width="0.1524" layer="91"/>
-<wire x1="93.98" y1="116.84" x2="81.28" y2="116.84" width="0.1524" layer="91"/>
-<wire x1="81.28" y1="116.84" x2="81.28" y2="109.22" width="0.1524" layer="91"/>
-<junction x="93.98" y="116.84"/>
-<pinref part="IC1" gate="G$1" pin="PB6(XTAL1/TOSC1)"/>
-<pinref part="Y1" gate="G$1" pin="2"/>
-<pinref part="C2" gate="G$1" pin="1"/>
-</segment>
-</net>
-<net name="XTAL2" class="0">
-<segment>
-<wire x1="101.6" y1="111.76" x2="93.98" y2="111.76" width="0.1524" layer="91"/>
-<wire x1="93.98" y1="111.76" x2="91.44" y2="111.76" width="0.1524" layer="91"/>
-<wire x1="91.44" y1="111.76" x2="91.44" y2="109.22" width="0.1524" layer="91"/>
-<junction x="93.98" y="111.76"/>
-<pinref part="IC1" gate="G$1" pin="PB7(XTAL2/TOSC2)"/>
-<pinref part="Y1" gate="G$1" pin="1"/>
-<pinref part="C1" gate="G$1" pin="1"/>
-</segment>
-</net>
